Commit message: Xacro wheel orientation corrected

File: install/rc_sim_description/share/rc_sim_description/urdf/rc_car.urdf.xacro (robot description, xacro)
@@ -36,5 +36,5 @@
       </inertial>
       <visual>
-        <origin xyz="0 0 0" rpy="0 1.5708 0"/>
+        <origin xyz="0 0 0" rpy="1.5708 0 0"/>
         <geometry>
           <cylinder radius="${wheel_radius}" length="${wheel_thickness}"/>
@@ -43,5 +43,5 @@
       </visual>
       <collision>
-        <origin xyz="0 0 0" rpy="0 1.5708 0"/>
+        <origin xyz="0 0 0" rpy="1.5708 0 0"/>
         <geometry>
           <cylinder radius="${wheel_radius}" length="${wheel_thickness}"/>

Commit message: Implement rear-wheel drive control and Ackermann steering

File: install/rc_sim_description/share/rc_sim_description/urdf/rc_car.urdf.xacro (robot description, xacro)
@@ -5,4 +5,5 @@
   <xacro:property name="chassis_width" value="0.28"/>
   <xacro:property name="chassis_height" value="0.10"/>
+  <xacro:property name="chassis_clearance" value="0.03"/>
   <xacro:property name="wheel_radius" value="0.06"/>
   <xacro:property name="wheel_thickness" value="0.03"/>
@@ -94,10 +95,10 @@
   <link name="base_link">
     <inertial>
-      <origin xyz="0 0 ${chassis_height / 2.0}" rpy="0 0 0"/>
+      <origin xyz="0 0 ${chassis_height / 2.0 + chassis_clearance}" rpy="0 0 0"/>
       <mass value="${chassis_mass}"/>
       <inertia ixx="${chassis_ixx}" ixy="0.0" ixz="0.0" iyy="${chassis_iyy}" iyz="0.0" izz="${chassis_izz}"/>
     </inertial>
     <visual>
-      <origin xyz="0 0 ${chassis_height / 2.0}" rpy="0 0 0"/>
+      <origin xyz="0 0 ${chassis_height / 2.0 + chassis_clearance}" rpy="0 0 0"/>
       <geometry>
         <box size="${chassis_length} ${chassis_width} ${chassis_height}"/>
@@ -106,5 +107,5 @@
     </visual>
     <collision>
-      <origin xyz="0 0 ${chassis_height / 2.0}" rpy="0 0 0"/>
+      <origin xyz="0 0 ${chassis_height / 2.0 + chassis_clearance}" rpy="0 0 0"/>
       <geometry>
         <box size="${chassis_length} ${chassis_width} ${chassis_height}"/>
@@ -123,3 +124,37 @@
     <kd>20.0</kd>
   </gazebo>
+  <gazebo>
+    <plugin
+      filename="gz-sim-joint-controller-system"
+      name="gz::sim::systems::JointController">
+      <joint_name>rear_left_wheel_joint</joint_name>
+    </plugin>
+    <plugin
+      filename="gz-sim-joint-controller-system"
+      name="gz::sim::systems::JointController">
+      <joint_name>rear_right_wheel_joint</joint_name>
+    </plugin>
+    <plugin
+      filename="gz-sim-joint-position-controller-system"
+      name="gz::sim::systems::JointPositionController">
+      <joint_name>front_left_wheel_steer_joint</joint_name>
+      <topic>/model/rc_car/joint/front_left_wheel_steer_joint/cmd_pos</topic>
+      <p_gain>20.0</p_gain>
+      <i_gain>0.1</i_gain>
+      <d_gain>0.5</d_gain>
+      <cmd_max>0.6</cmd_max>
+      <cmd_min>-0.6</cmd_min>
+    </plugin>
+    <plugin
+      filename="gz-sim-joint-position-controller-system"
+      name="gz::sim::systems::JointPositionController">
+      <joint_name>front_right_wheel_steer_joint</joint_name>
+      <topic>/model/rc_car/joint/front_right_wheel_steer_joint/cmd_pos</topic>
+      <p_gain>20.0</p_gain>
+      <i_gain>0.1</i_gain>
+      <d_gain>0.5</d_gain>
+      <cmd_max>0.6</cmd_max>
+      <cmd_min>-0.6</cmd_min>
+    </plugin>
+  </gazebo>
 </robot>

Commit message: Lidar implemented

File: install/rc_sim_description/share/rc_sim_description/urdf/rc_car.urdf.xacro (robot description, xacro)
@@ -113,8 +113,82 @@
     </collision>
   </link>
+  <link name="lidar_link">
+    <inertial>
+      <origin xyz="0 0 0" rpy="0 0 0"/>
+      <mass value="0.05"/>
+      <inertia ixx="0.0001" ixy="0.0" ixz="0.0" iyy="0.0001" iyz="0.0" izz="0.0001"/>
+    </inertial>
+    <visual>
+      <origin xyz="0 0 0" rpy="0 0 0"/>
+      <geometry>
+        <cylinder radius="0.02" length="0.03"/>
+      </geometry>
+      <material name="chassis_grey"/>
+    </visual>
+  </link>
+  <joint name="lidar_joint" type="fixed">
+    <parent link="base_link"/>
+    <child link="lidar_link"/>
+    <origin xyz="${chassis_length/2 - 0.05} 0 ${chassis_height/2 + 0.08}" rpy="0 0 0"/>
+  </joint>
+  <gazebo reference="lidar_link">
+    <sensor name="lidar" type="gpu_lidar">
+      <always_on>true</always_on>
+      <update_rate>12</update_rate>
+      <visualize>true</visualize>
+      <topic>/scan</topic>
+      <lidar>
+        <scan>
+          <horizontal>
+            <samples>360</samples>
+            <resolution>1</resolution>
+            <min_angle>-3.14159265</min_angle>
+            <max_angle>3.14159265</max_angle>
+          </horizontal>
+        </scan>
+        <range>
+          <min>0.05</min>
+          <max>12.0</max>
+          <resolution>0.01</resolution>
+        </range>
+        <noise type="gaussian">
+          <mean>0.0</mean>
+          <stddev>0.0</stddev>
+        </noise>
+      </lidar>
+    </sensor>
+  </gazebo>
   <xacro:steered_wheel name="front_left_wheel" parent="base_link" xyz="${wheel_base_x} ${wheel_track_y} ${axle_height}"/>
   <xacro:steered_wheel name="front_right_wheel" parent="base_link" xyz="${wheel_base_x} ${-wheel_track_y} ${axle_height}"/>
   <xacro:wheel name="rear_left_wheel" parent="base_link" xyz="${-wheel_base_x} ${wheel_track_y} ${axle_height}"/>
   <xacro:wheel name="rear_right_wheel" parent="base_link" xyz="${-wheel_base_x} ${-wheel_track_y} ${axle_height}"/>
+  <ros2_control name="rc_car_system" type="system">
+    <hardware>
+      <plugin>gazebo_ros2_control/GazeboSystem</plugin>
+    </hardware>
+    <joint name="rear_left_wheel_joint">
+      <command_interface name="velocity"/>
+      <state_interface name="position"/>
+      <state_interface name="velocity"/>
+    </joint>
+    <joint name="rear_right_wheel_joint">
+      <command_interface name="velocity"/>
+      <state_interface name="position"/>
+      <state_interface name="velocity"/>
+    </joint>
+    <joint name="front_left_wheel_steer_joint">
+      <command_interface name="position"/>
+      <state_interface name="position"/>
+      <state_interface name="velocity"/>
+    </joint>
+    <joint name="front_right_wheel_steer_joint">
+      <command_interface name="position"/>
+      <state_interface name="position"/>
+      <state_interface name="velocity"/>
+    </joint>
+  </ros2_control>
+  <gazebo>
+    <plugin name="gazebo_ros2_control" filename="libgazebo_ros2_control.so"/>
+  </gazebo>
   <gazebo reference="base_link">
     <material>Gazebo/Grey</material>

Commit message: simulation with movement algorithm ackerman model dynamics

File: install/rc_sim_description/share/rc_sim_description/urdf/rc_car.urdf.xacro (robot description, xacro)
@@ -54,5 +54,5 @@
       <child link="${name}"/>
       <origin xyz="${xyz}" rpy="1.5708 0 0"/>
-      <axis xyz="0 0 1"/>
+      <axis xyz="0 0 -1"/>
     </joint>
     <gazebo reference="${name}">

Commit message: camera simul added and implementation of image_viewer

File: install/rc_sim_description/share/rc_sim_description/urdf/rc_car.urdf.xacro (robot description, xacro)
@@ -127,8 +127,27 @@
     </visual>
   </link>
+  <link name="camera_link">
+    <inertial>
+      <origin xyz="0 0 0" rpy="0 0 0"/>
+      <mass value="0.05"/>
+      <inertia ixx="0.0001" ixy="0.0" ixz="0.0" iyy="0.0001" iyz="0.0" izz="0.0001"/>
+    </inertial>
+    <visual>
+      <origin xyz="0 0 0" rpy="0 0 0"/>
+      <geometry>
+        <box size="0.04 0.02 0.02"/>
+      </geometry>
+      <material name="chassis_grey"/>
+    </visual>
+  </link>
   <joint name="lidar_joint" type="fixed">
     <parent link="base_link"/>
     <child link="lidar_link"/>
     <origin xyz="${chassis_length/2 - 0.05} 0 ${chassis_height/2 + 0.08}" rpy="0 0 0"/>
+  </joint>
+  <joint name="camera_joint" type="fixed">
+    <parent link="base_link"/>
+    <child link="camera_link"/>
+    <origin xyz="0.25 0.0 0.20" rpy="0 0 0"/>
   </joint>
   <gazebo reference="lidar_link">
@@ -159,4 +178,26 @@
     </sensor>
   </gazebo>
+  <gazebo reference="camera_link">
+    <sensor name="camera" type="camera">
+      <always_on>true</always_on>
+      <update_rate>30</update_rate>
+      <visualize>false</visualize>
+      <topic>/camera/image_raw</topic>
+      <camera>
+        <horizontal_fov>1.047</horizontal_fov>
+        <image>
+          <width>640</width>
+          <height>480</height>
+          <format>R8G8B8</format>
+        </image>
+        <clip>
+          <near>0.05</near>
+          <far>50.0</far>
+        </clip>
+      </camera>
+      <frame_id>camera_link</frame_id>
+      <camera_info_topic>/camera/camera_info</camera_info_topic>
+    </sensor>
+  </gazebo>
   <xacro:steered_wheel name="front_left_wheel" parent="base_link" xyz="${wheel_base_x} ${wheel_track_y} ${axle_height}"/>
   <xacro:steered_wheel name="front_right_wheel" parent="base_link" xyz="${wheel_base_x} ${-wheel_track_y} ${axle_height}"/>
