Commit message: feat(sim): the car identifies its own plant and drives on it
The simulated driver assumed it knew itself: the wheelbase, where its axles
are, the gain and centre of its servo, the map from a speed command to a
speed, and where its LiDAR is mounted all came from vehicle.yaml. On the real
car none of those is measured, so the controller now measures them, from the
only sensor it has: the trained odometry.

Three aggregates are identifiable from one pose increment per revolution, and
they are the three the control needs. The lever arm comes out of an exact
identity -- dy - dx tan(dyaw/2) = 2 tan(dyaw/2) arm, with the curvature
cancelling for any turn angle -- and replaces rear_offset_m, answering at once
how far the front axle is and where the LiDAR sits. The curvature map (a gain
per side, a trim, a v^2 term for the slip of the rear axle) absorbs the
wheelbase, the servo and the linkage, and the wheelbase cancels on the way out
rather than being estimated. The speed map carries the state of the battery in
a gain that is a random walk, with the motor's start threshold bracketed from
the launches instead of fitted through its kink.

Every estimate starts at the datasheet with the datasheet's covariance, so a
car that has learned nothing publishes what it published before, and nothing
moves in a direction nothing excited. A floor under the measurement variance
(the residual measured on recorded runs) keeps the sub-millimetre published
sigmas from making it overconfident, and a watchdog restores the datasheet if
the identified model ever predicts worse. The confidence it reaches is
one-sided: it only ever asks for less speed, less grip, more margin and a
longer lookahead than the nominal configuration.

The car also gets out of places it used to stop in for good: it creeps forward
where the lane is proven and backs out, over ground it has already driven,
where it is not.

To validate any of this honestly a run has to draw its own plant, because with
nothing to find the identification buys about 4 % of residual and proves
nothing. draw_plant_mismatch draws it from the same spread the estimator
carries as its prior; every key defaults to the identity, so the pose dataset
is untouched, and what came up goes to run_config.json for the evaluation
only, with the firewall forbidding the car side from reading it.

Two defects found on the way: rc_car.urdf.xacro placed both axles at
+-front_axle_offset_x, which is symmetric about base_link and so only agreed
with wheelbase_m at the nominal values; and sim_actuation_node froze the
steering below 0.05 m/s, losing it exactly where a car manoeuvres.

Validated in Gazebo in the configuration the car runs (polar ICP + ONNX) and in
the 2D harness over the documented seeds, where the drawn plant costs the
unmodified controller two runs out of ten and five seconds a lap.

Co-Authored-By: Claude Opus 5 <noreply@anthropic.com>

File: simulation/ros2_ws/src/rc_sim_description/urdf/rc_car.urdf.xacro (robot description, xacro)
@@ -43,4 +43,10 @@
   <xacro:arg name="imu_xyz" default=""/>
   <xacro:arg name="imu_rpy" default="0 0 0"/>
+  <!-- Geometry of the axles. The defaults are the nominal car; a real2sim run
+       draws them (pose_dataset.vehicle.draw_plant_mismatch) because the real
+       car's wheelbase and the position of its axles are not measured, and the
+       controller has to identify what it is driving. -->
+  <xacro:arg name="wheelbase_m" default="0.30"/>
+  <xacro:arg name="rear_axle_offset_x" default="-0.15"/>
   <!-- Basic dimensions -->
   <xacro:property name="chassis_length" value="0.46"/>
@@ -50,6 +56,6 @@
   <xacro:property name="wheel_radius" value="0.06"/>
   <xacro:property name="wheel_thickness" value="0.03"/>
-  <xacro:property name="wheelbase_m" value="0.30"/>
-  <xacro:property name="rear_axle_offset_x" value="-0.15"/>
+  <xacro:property name="wheelbase_m" value="$(arg wheelbase_m)"/>
+  <xacro:property name="rear_axle_offset_x" value="$(arg rear_axle_offset_x)"/>
   <xacro:property name="front_axle_offset_x" value="${rear_axle_offset_x + wheelbase_m}"/>
   <xacro:property name="steering_limit_rad" value="0.3141592654"/>
@@ -57,5 +63,9 @@
   <xacro:property name="lidar_offset_z" value="0.12"/>
   <!-- Placement helpers -->
-  <xacro:property name="wheel_base_x" value="${front_axle_offset_x}"/>
+  <!-- Each axle sits at its own offset. They used to share
+       front_axle_offset_x, which places both axles symmetrically about
+       base_link: with the nominal -0.15 / 0.30 the two agree and nothing shows,
+       but a car whose axles are not symmetric about its origin then had a
+       wheelbase of 2 * front_axle_offset_x instead of wheelbase_m. -->
   <xacro:property name="wheel_track_y" value="${chassis_width / 2.0 + wheel_thickness / 2.0 - 0.01}"/>
   <xacro:property name="axle_height" value="${wheel_radius}"/>
@@ -434,8 +444,8 @@
     </gazebo>
   </xacro:if>
-  <xacro:steered_wheel name="front_left_wheel" parent="base_link" xyz="${wheel_base_x} ${wheel_track_y} ${axle_height}"/>
-  <xacro:steered_wheel name="front_right_wheel" parent="base_link" xyz="${wheel_base_x} ${-wheel_track_y} ${axle_height}"/>
-  <xacro:wheel name="rear_left_wheel" parent="base_link" xyz="${-wheel_base_x} ${wheel_track_y} ${axle_height}"/>
-  <xacro:wheel name="rear_right_wheel" parent="base_link" xyz="${-wheel_base_x} ${-wheel_track_y} ${axle_height}"/>
+  <xacro:steered_wheel name="front_left_wheel" parent="base_link" xyz="${front_axle_offset_x} ${wheel_track_y} ${axle_height}"/>
+  <xacro:steered_wheel name="front_right_wheel" parent="base_link" xyz="${front_axle_offset_x} ${-wheel_track_y} ${axle_height}"/>
+  <xacro:wheel name="rear_left_wheel" parent="base_link" xyz="${rear_axle_offset_x} ${wheel_track_y} ${axle_height}"/>
+  <xacro:wheel name="rear_right_wheel" parent="base_link" xyz="${rear_axle_offset_x} ${-wheel_track_y} ${axle_height}"/>
   <gazebo reference="base_link">
     <material>Gazebo/Grey</material>
